File: batty_trees_test_pcb/_autosave-batty_trees_test_pcb.kicad_pcb (KiCad board)
At the start: 4 copper layers, 127 x 152.4 mm, 161 parts, among them J1 JSH_PH_B3B-PH-K, J10 Conn_02x04_Odd_Even, J11 Conn_02x08_Odd_Even, J12 Conn_02x04_Odd_Even, J13 OPAL_KELLY, J2 JSH_PH_B3B-PH-K, J3 Header, J4 Header, J5 Conn_02x04_Odd_Even, J6 UJC-HP-3-SMT-TR, J7 105-1102-001, J8 105-1103-001, J9 Conn_02x04_Odd_Even, U1 LMH6611, U10 LMH6611, U11 LMH6611, U12 LMH6611, U13 LT3042xMSE, U14 LT3042xMSE, U15 LT3042xMSE, U16 AD8031, U17 LTC1844ES5-3.3, U2 LMH6611, U3 LMH6611, U4 LMH6611, U5 LMH6611, U6 LMH6611, U7 LMH6611, U8 LMH6611, U9 LMH6611, X1 PLCC_84

Commit message: Layout finished and gerbers generated checking for DFM
Routing:
- net /rst: track 140.3 -> 139.3 mm
Changed lines of the file:
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@@
     (pcbplotparams
       (layerselection 0x010fc_ffffffff)
-      (usegerberextensions false)
+      (usegerberextensions true)
       (usegerberattributes false)
       (usegerberadvancedattributes false)
@@
       (psa4output false)
       (plotreference true)
-      (plotvalue true)
+      (plotvalue false)
       (plotinvisibletext false)
       (padsonsilk false)
@@
       (outputformat 1)
       (mirror false)
-      (drillshape 1)
+      (drillshape 0)
       (scaleselection 1)
-      (outputdirectory ""))
+      (outputdirectory "gerbers/"))
   )
   (net 0 "")
@@
   (segment (start 96.52 49.53) (end 97.79 50.8) (width 0.25) (layer B.Cu) (net 88))
   (segment (start 97.79 50.8) (end 97.79 73.406) (width 0.25) (layer B.Cu) (net 88))
-  (segment (start 97.79 73.406) (end 97.79 81.153) (width 0.25) (layer B.Cu) (net 88))
-  (segment (start 98.132002 81.153) (end 103.212002 86.233) (width 0.25) (layer B.Cu) (net 88))
-  (segment (start 97.79 81.153) (end 98.132002 81.153) (width 0.25) (layer B.Cu) (net 88))
-  (segment (start 103.212002 86.233) (end 105.156 86.233) (width 0.25) (layer B.Cu) (net 88))
-  (segment (start 105.156 86.233) (end 108.077 89.154) (width 0.25) (layer B.Cu) (net 88))
-  (segment (start 106.034999 91.196001) (end 106.034999 102.880001) (width 0.25) (layer B.Cu) (net 88))
-  (segment (start 108.077 89.154) (end 106.034999 91.196001) (width 0.25) (layer B.Cu) (net 88))
   (via (at 103.632 112.014) (size 0.8) (drill 0.4) (layers F.Cu B.Cu) (net 88))
-  (segment (start 106.034999 102.880001) (end 103.632 105.283) (width 0.25) (layer B.Cu) (net 88))
-  (segment (start 103.632 105.283) (end 103.632 112.014) (width 0.25) (layer B.Cu) (net 88))
   (segment (start 105.789 112.014) (end 105.8 112.025) (width 0.25) (layer F.Cu) (net 88))
   (segment (start 103.632 112.014) (end 105.789 112.014) (width 0.25) (layer F.Cu) (net 88))
@@
   (segment (start 124.299 146.177) (end 127.601 149.479) (width 0.25) (layer B.Cu) (net 88))
   (segment (start 106.934 146.177) (end 124.299 146.177) (width 0.25) (layer B.Cu) (net 88))
+  (segment (start 97.79 82.4865) (end 97.79 81.0895) (width 0.25) (layer B.Cu) (net 88))
+  (segment (start 99.5045 84.201) (end 97.79 82.4865) (width 0.25) (layer B.Cu) (net 88))
+  (segment (start 102.743 84.201) (end 99.5045 84.201) (width 0.25) (layer B.Cu) (net 88))
+  (segment (start 106.034999 87.492999) (end 102.743 84.201) (width 0.25) (layer B.Cu) (net 88))
+  (segment (start 97.79 81.0895) (end 97.79 81.153) (width 0.25) (layer B.Cu) (net 88))
+  (segment (start 103.632 112.014) (end 103.632 105.283) (width 0.25) (layer B.Cu) (net 88))
+  (segment (start 106.034999 102.880001) (end 106.034999 87.492999) (width 0.25) (layer B.Cu) (net 88))
+  (segment (start 97.79 73.406) (end 97.79 81.0895) (width 0.25) (layer B.Cu) (net 88))
+  (segment (start 103.632 105.283) (end 106.034999 102.880001) (width 0.25) (layer B.Cu) (net 88))
   (segment (start 72.9461 111.2564) (end 74.168 110.0345) (width 0.25) (layer F.Cu) (net 89))
   (segment (start 71.9722 111.2564) (end 72.9461 111.2564) (width 0.25) (layer F.Cu) (net 89))
