File: batty_trees_test_pcb/batty_trees_test_pcb.kicad_pcb (KiCad board)
At the start: 4 copper layers, 127 x 152.4 mm, 134 parts, among them J1 JSH_PH_B3B-PH-K, J2 JSH_PH_B3B-PH-K, J3 Header, J4 Header, J5 OPAL_KELLY, J6 UJC-HP-3-SMT-TR, J7 105-1102-001, J8 105-1103-001, U1 LMH6611, U10 LMH6611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

Commit message: more layout work ~90% finished
Parts:
- added C22: 0.1uF, Capacitor_SMD:C_0805_2012Metric_Pad1.15x1.40mm_HandSolder, F.Cu at (146.4, 41.4)
- added C23: 0.1uF, Capacitor_SMD:C_0805_2012Metric_Pad1.15x1.40mm_HandSolder, F.Cu at (50.0, 44.1)
- added C24: 0.1uF, Capacitor_SMD:C_0805_2012Metric_Pad1.15x1.40mm_HandSolder, F.Cu at (60.3, 39.8)
- added C25: 0.1uF, Capacitor_SMD:C_0805_2012Metric_Pad1.15x1.40mm_HandSolder, F.Cu at (125.2, 39.8)
- added C26: 0.1uF, Capacitor_SMD:C_0805_2012Metric_Pad1.15x1.40mm_HandSolder, F.Cu at (56.4, 39.8)
- added C27: 0.1uF, Capacitor_SMD:C_0805_2012Metric_Pad1.15x1.40mm_HandSolder, F.Cu at (121.4, 39.8)
- added C28: 0.1uF, Capacitor_SMD:C_0805_2012Metric_Pad1.15x1.40mm_HandSolder, F.Cu at (57.5, 8.13)
- added C29: 0.1uF, Capacitor_SMD:C_0805_2012Metric_Pad1.15x1.40mm_HandSolder, F.Cu at (67.8, 44.1)
- added C30: 0.1uF, Capacitor_SMD:C_0805_2012Metric_Pad1.15x1.40mm_HandSolder, F.Cu at (57.5, 11.1)
- added C31: 0.1uF, Capacitor_SMD:C_0805_2012Metric_Pad1.15x1.40mm_HandSolder, F.Cu at (62.3, 8.13)
- added C32: 0.1uF, Capacitor_SMD:C_0805_2012Metric_Pad1.15x1.40mm_HandSolder, F.Cu at (115.1, 44.1)
- added C33: 0.1uF, Capacitor_SMD:C_0805_2012Metric_Pad1.15x1.40mm_HandSolder, F.Cu at (62.3, 11.1)
- added C34: 0.1uF, Capacitor_SMD:C_0805_2012Metric_Pad1.15x1.40mm_HandSolder, F.Cu at (132.8, 44.1)
- added J10: Conn_02x04_Odd_Even, Connector_PinHeader_2.54mm:PinHeader_2x04_P2.54mm_Vertical, F.Cu at (127.0, 67.1)
- added J11: Conn_02x08_Odd_Even, Connector_PinHeader_2.54mm:PinHeader_2x08_P2.54mm_Vertical, F.Cu at (49.0, 57.1)
- added J12: Conn_02x04_Odd_Even, Connector_PinHeader_2.54mm:PinHeader_2x04_P2.54mm_Vertical, F.Cu at (127.0, 56.9)
- added J5: Conn_02x04_Odd_Even, Connector_PinHeader_2.54mm:PinHeader_2x04_P2.54mm_Vertical, F.Cu at (96.5, 91.4)
- added J9: Conn_02x04_Odd_Even, Connector_PinHeader_2.54mm:PinHeader_2x04_P2.54mm_Vertical, F.Cu at (79.2, 91.4)
- added MH1: MountingHole_2.7mm_M2.5, MountingHole:MountingHole_2.7mm_M2.5, F.Cu at (28.4, 174.8)
- added MH2: MountingHole_2.7mm_M2.5, MountingHole:MountingHole_2.7mm_M2.5, F.Cu at (149.4, 174.8)
- added MH3: MountingHole_2.7mm_M2.5, MountingHole:MountingHole_2.7mm_M2.5, F.Cu at (149.4, 28.4)
- added MH4: MountingHole_2.7mm_M2.5, MountingHole:MountingHole_2.7mm_M2.5, F.Cu at (28.4, 28.4)
- moved R46 228.9 mm to (34.3, 163.1), turned to 90 degrees
- moved C5 219.2 mm to (33.8, 70.9), turned to 180 degrees
- moved R39 216.5 mm to (33.5, 77.5), turned to 90 degrees
- moved C7 212.8 mm to (33.5, 49.1), turned to 180 degrees
- moved C8 212.2 mm to (35.8, 77.5), turned to 90 degrees
- moved TP12 209.1 mm to (37.7, 48.6)
- moved C13 208.9 mm to (39.0, 51.9), turned to 270 degrees
- moved TP13 207.9 mm to (37.8, 70.6)
- moved C10 207.7 mm to (34.5, 55.9), turned to 90 degrees
- moved C3 207.0 mm to (53.6, 166.1), turned to 90 degrees
- moved C16 206.2 mm to (41.1, 51.9), turned to 270 degrees
- moved R41 205.6 mm to (32.0, 55.9), turned to 90 degrees
- moved C2 205.3 mm to (51.3, 166.1), turned to 270 degrees
- moved R47 204.1 mm to (36.6, 163.1), turned to 90 degrees
- moved R25 200.9 mm to (52.6, 44.1), turned to 90 degrees
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- renumbered J5 to J13, R12 to Re
Connections:
- J13 pad 115: Net-(J5-Pad115) -> VDD
- J13 pad 135: Net-(J5-Pad135) -> VDD
- JP5 pad 1: /Power/DD_VREF_REGOUT -> Net-(JP5-Pad1)
- JP5 pad 2: Net-(JP5-Pad2) -> /dd_vref
- R42 pad 1: Net-(JP5-Pad2) -> /Power/DD_VREF_REGOUT
- R42 pad 2: /dd_vref -> Net-(JP5-Pad1)
Routing:
- net GND: track 19.0 -> 107.7 mm, vias 13 -> 80
- net +3V3: track 0.00 -> 37.0 mm, vias 0 -> 38
- net /l_vpulse3: track 78.7 -> 109.2 mm
- net /l_vpulse1: track 84.1 -> 113.6 mm
- net /l_slow_data_out: track 89.2 -> 117.7 mm
- net /l_vpulse4: track 72.8 -> 100.8 mm
- net /r_vpulse7: track 57.6 -> 85.4 mm
- net /l_slow_clk: track 94.2 -> 121.6 mm
- net /l_vpulse2: track 78.2 -> 105.2 mm
- net /r_vpulse5: track 62.0 -> 88.7 mm
- net /l_slow_valid_out: track 83.2 -> 109.1 mm
- net /r_vpulse3: track 67.6 -> 93.3 mm
- net /r_vpulse1: track 72.9 -> 98.3 mm
- net /r_vpulse8: track 51.3 -> 76.6 mm
- net /l_slow_data_load: track 88.7 -> 113.5 mm
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- added copper zone on F.Cu, net +3V3
- added copper zone on In2.Cu, net +3V3
- added copper zone on F.Cu, net /Power/VDDA_REGOUT
- added copper zone on F.Cu, net /Power/VDD_REGOUT
- added copper zone on In1.Cu, net GND
- added copper zone on F.Cu, net VDC
- added copper zone on In2.Cu, net VDC
- added copper zone on In2.Cu, net VDD
- added copper zone on In2.Cu, net VDDA
- removed copper zone on In2.Cu, net GND
Other:
- board text added: "GND"
- board text added: "VDC"
- board text added: "VDD"
- board text added: "VDDA"
- board text added: "VREF"

Commit message: Layout finished and gerbers generated checking for DFM
Parts:
- added C35: 0.1uF, Capacitor_SMD:C_0805_2012Metric_Pad1.15x1.40mm_HandSolder, F.Cu at (122.8, 142.2)
- added G***: LOGO, OSU_SIM_BASIC:LOGOmed, F.Cu at (39.5, 109.0)
- added R52: 1k, Resistor_SMD:R_0805_2012Metric_Pad1.15x1.40mm_HandSolder, F.Cu at (120.4, 142.2)
- added R53: 100k, Resistor_SMD:R_0805_2012Metric_Pad1.15x1.40mm_HandSolder, F.Cu at (125.2, 142.2)
- added S1: GPTS203211B, digikey-footprints:PushButton_12x12mm_THT_GPTS203211B, F.Cu at (122.3, 149.5)
- moved R31 175.2 mm to (78.5, 39.2), turned to 180 degrees
- moved R35 166.2 mm to (78.5, 33.7)
- moved TP5 166.2 mm to (74.2, 31.4)
- moved R37 151.0 mm to (82.7, 33.7), turned to 180 degrees
- moved U10 148.6 mm to (86.9, 36.4)
- moved R29 146.5 mm to (86.7, 39.2), turned to 180 degrees
- moved R32 144.2 mm to (98.8, 39.4), turned to 180 degrees
- moved U9 144.2 mm to (78.5, 36.4)
- moved JP1 143.3 mm to (74.2, 35.6)
- moved R33 139.4 mm to (86.9, 33.7)
- moved R36 139.1 mm to (98.8, 33.8)
- moved U11 136.1 mm to (98.8, 36.6)
- moved TP6 134.3 mm to (94.7, 31.4)
- moved R34 133.8 mm to (106.9, 33.8)
- moved R30 131.9 mm to (106.9, 39.4)
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- renumbered Re to R12
Connections:
- J13 pad 151: Net-(J13-Pad151) -> /rst
- J6 pad S1: GND -> Net-(J6-PadS1)
- J6 pad S2: GND -> Net-(J6-PadS2)
- J6 pad S3: GND -> Net-(J6-PadS3)
- J6 pad S4: GND -> Net-(J6-PadS4)
Routing:
- net /rst: track 0.00 -> 139.3 mm, vias 0 -> 1
- net /rate_crtl: track 66.4 -> 177.4 mm
- net /ser_test: track 84.8 -> 181.9 mm
- net /dd_pulse_width8: track 38.9 -> 119.6 mm
- net /mux_sel: track 72.4 -> 145.4 mm
- net /dd_lin: track 0.00 -> 51.5 mm
- net /l_vinn: track 2.40 -> 42.0 mm
- net /dd_rin: track 0.00 -> 38.7 mm
- net /dd_vref: track 0.00 -> 38.6 mm
- net /r_vinp: track 0.00 -> 36.1 mm
- net /AFE/R_VIN_BUFP: track 22.5 -> 48.9 mm, vias 0 -> 1
- net /r_vinn: track 2.40 -> 27.7 mm
- net /VMID: track 0.00 -> 25.1 mm, vias 0 -> 8
- net /AFE/R_VIN_BUFN: track 20.1 -> 45.0 mm
- net /l_vinp: track 2.40 -> 26.9 mm
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- added copper zone on B.Cu, net /VMID
Other:
- board text added: "+5V"
- board text added: "DD_PULSE_WIDTH8"
- board text added: "GND dd_valid GND dd_latch_out GND dd_clk GND dd_dir"
- board text added: "GND l_vpulse8 GND l_vpulse7 GND l_vpulse6 GND l_vpulse5"
- board text added: "GND r_vpulse1 GND r_vpulse2 GND r_vpulse3 GND r_vpulse4 GND r_vpulse5 GND r_vpulse6 GND r_vpulse7 GND r_vpulse8"
- board text added: "KiCAD files found at https://github.com/clocktop/batty_trees_test_pcb"
- board text added: "Kyle Clocker 09/2020 kyleclocker.com"
- board text added: "L_VIN_BUF + G -"
- board text added: "MUX_SEL"
- board text added: "OSU SIM LAB"
- board text added: "R chan + G -"
- board text added: "RATE_CRTL"
- board text added: "RST"
- board text added: "R_VIN_BUF + G -"
- board text added: "SER_TEST"
- board text added: "TSMC JUNE 2020 Test"
- board text added: "VDD Adj"
- board text added: "VDDA Adj"
- board text added: "VMID Adj"
- board text added: "VREF Adj"
- board text added: "dd_lin"
- board text added: "dd_rin"
- board text added: "l_chan + G -"
- board text added: "l_slow_clk GND l_slow_data_load GND l_slow_data_out GND l_slow_valid_out GND"
- board text added: "l_vinn"
- board text added: "l_vinp"
- board text added: "l_vpulse1 GND l_vpulse2 GND l_vpulse3 GND l_vpulse4 GND"
- board text added: "r_vinn"
- board text added: "r_vinp"
